File: kicad/DiscoDongle.kicad_pcb (KiCad board)
At the start: 2 copper layers, 58.4 x 15.9 mm, 22 parts, among them J1 USB_B, J2 RJ45, U1 FT232RL, U2 ISL81487E

Commit message: Rename board
Other:
- board text added: "DiscoDongle"
- board text removed: "DiscoDongle2"
Changed lines of the file:
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@@
-(kicad_pcb (version 4) (host pcbnew 4.0.2-stable)
+(kicad_pcb (version 4) (host pcbnew 4.0.4-stable)
   (general
     (links 53)
     (no_connects 2)
-    (area 136.403599 97.104999 196.308401 113.9214)
+    (area 136.403599 97.104999 196.308401 114.0214)
     (thickness 1.6)
     (drawings 6)
@@
     (34 B.Paste user)
     (35 F.Paste user)
-    (36 B.SilkS user hide)
+    (36 B.SilkS user)
     (37 F.SilkS user)
     (38 B.Mask user)
@@
     (effects (font (size 1.2 1.2) (thickness 0.2)) (justify mirror))
   )
-  (gr_text DiscoDongle2 (at 166.37 108.331 180) (layer B.SilkS)
+  (gr_text DiscoDongle (at 166.37 108.331 180) (layer B.SilkS)
     (effects (font (size 1.8 1.8) (thickness 0.3)) (justify mirror))
   )

Commit message: Change USB to micro-B. Add part numbers
Parts:
- J1: value USB_B -> USB_B_Micro; footprint Connect:USB_B -> DongleParts:USB_Micro-B
- moved REF*** 10.8 mm to (168.5, 100.6)
- moved J1 10.5 mm to (141.4, 105.1), turned to 90 degrees
- moved C1 8.21 mm to (151.9, 101.3)
- moved C2 8.21 mm to (151.9, 103.5)
- moved C3 8.21 mm to (151.9, 105.8)
- moved C4 8.21 mm to (151.9, 108.1)
Connections:
- J1 pad 4: GND -> Net-(J1-Pad4)
Routing:
- net Net-(J1-Pad2): track 15.8 -> 24.5 mm, vias 0 -> 1
- net Net-(C4-Pad1): track 23.6 -> 15.2 mm
- net Net-(J1-Pad3): track 18.2 -> 24.2 mm, vias 0 -> 1
- net Signal: track 23.9 -> 26.3 mm
- net GND: track 0.00 -> 1.20 mm
- net +5V: track 17.5 -> 18.3 mm, vias 8 -> 7
Other:
- board text added: "2016 - rev7"
- board text added: "A/Y"
- board text added: "B/Z"
- board text added: "D"
- board text added: "G"
- board text added: "S"
- board text removed: "2016 - rev6"

Commit message: Micro USB
Parts:
- D3: value D -> Daisy
- D4: value S -> Signal
- moved J1 7.63 mm to (149.0, 105.1)
- moved C3 6.51 mm to (148.7, 111.5), turned to 0 degrees
- moved C2 4.66 mm to (152.2, 98.9), turned to 0 degrees
- moved C1 4.15 mm to (148.5, 98.9)
- moved C4 3.42 mm to (152.4, 111.5)
Routing:
- net Net-(J1-Pad2): track 24.5 -> 16.8 mm
- net Net-(J1-Pad3): track 24.2 -> 16.9 mm
- net GND: track 1.20 -> 4.95 mm
- net +5V: track 18.3 -> 14.9 mm, vias 7 -> 9
- net Net-(C4-Pad1): track 15.2 -> 17.0 mm
Other:
- board size 58.4 x 15.9 mm -> 49.4 x 15.8 mm
- net class Default: clearance 0.1524 -> 0.16
- rule trace_clearance: 0.1524 -> 0.16
